File: MainBoard/_autosave-VertexBot.kicad_pcb (KiCad board)
At the start: 2 copper layers, 115.6 x 107.8 mm, 47 parts, among them J1 Battery, J4 Left Motor, J5 Right Motor, J6 Led Strip, Q1 BSS138, Q2 BSS138, Q3 BSS138, SW1 SW_SPST, U1 DRV8830DGQR, U10 MAX4466, U11 MAX4466, U12 ESP32-S3-CAM-B, U13 ESP32-S3-CAM-A, U14 MAX98357A, U2 DRV8830DGQR, U3 S13V30F5, U5 INMP441, U6 0.96 INCH OLED, U7 DRV5033AJxLPG, U8 DRV5033AJxLPG, U9 MPU 6050

Commit message: Footprints complete and rough test placement on the board
Changed lines of the file:
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@@
 		)
 		(property "Value" "MAX4466"
-			(at 0 7.85 0)
+			(at 0 8.89 0)
 			(layer "F.Fab")
 			(effects
@@
 			(layer "F.Fab")
 		)
+		(fp_text user "MAX4466"
+			(at -3.429 9.4742 0)
+			(unlocked yes)
+			(layer "F.SilkS")
+			(effects
+				(font
+					(size 1 1)
+					(thickness 0.1)
+				)
+				(justify left bottom)
+			)
+		)
 		(fp_text user "${REFERENCE}"
 			(at 0 2.54 90)
@@
 		)
 		(property "Value" "MAX4466"
-			(at 0 7.85 0)
+			(at -0.0762 8.5344 0)
 			(layer "F.Fab")
 			(effects
@@
 			(layer "F.Fab")
 		)
+		(fp_text user "MAX4466"
+			(at -3.4798 9.0932 0)
+			(unlocked yes)
+			(layer "F.SilkS")
+			(effects
+				(font
+					(size 1 1)
+					(thickness 0.1)
+				)
+				(justify left bottom)
+			)
+		)
 		(fp_text user "${REFERENCE}"
 			(at 0 2.54 90)
@@
 			(layer "F.Fab")
 		)
+		(fp_text user "INMP441"
+			(at 0.2032 8.0772 0)
+			(unlocked yes)
+			(layer "F.SilkS")
+			(effects
+				(font
+					(size 1 1)
+					(thickness 0.1)
+				)
+				(justify left bottom)
+			)
+		)
 		(fp_text user "${REFERENCE}"
